Commit message: Add digit mesh and modify urdf file to put 3 digits on the right hand. The posiitons are not tuned for the grasping

File: urdf/ergoCub/robots/ergoCubGazeboV1/model.urdf (robot description, URDF)
Before this commit: robot ergoCub, 169 links, 168 joints
Links:
- link r_hand_index_3: geometry collision mesh filename=package://ergoCub/meshes/simmechanics/digit.STL scale=1 1 1; visual mesh filename=package://ergoCub/meshes/simmechanics/digit.STL scale=1 1 1
- link r_hand_middle_2: geometry collision mesh filename=package://ergoCub/meshes/simmechanics/digit.STL scale=1 1 1; visual mesh filename=package://ergoCub/meshes/simmechanics/digit.STL scale=1 1 1
- link r_hand_thumb_3: geometry collision mesh filename=package://ergoCub/meshes/simmechanics/digit.STL scale=1 1 1; visual mesh filename=package://ergoCub/meshes/simmechanics/digit.STL scale=1 1 1
Joints:
- joint r_index_dist: origin xyz=0 -0.0014998229561488108 -0.030000484918389303 rpy=0 0 0 -> xyz=0 -0.0014998229561488108 -0.030000484918389303 rpy=3.14 0 -1.57
- joint r_middle_dist: origin xyz=1.3550151000546462e-07 -0.0014995238274964628 -0.03000020325318492 rpy=-0.0018721728628663644 0 -2.576685250299645e-07 -> xyz=1.3550151000546462e-07 -0.0014995238274964628 -0.03000020325318492 rpy=3.14 0 -1.57
- joint r_thumb_dist: origin xyz=0.019999518753341633 -0.0014995177497797996 -3.909354686637556e-07 rpy=0 0 0 -> xyz=0.019999518753341633 -0.0014995177497797996 -3.909354686637556e-07 rpy=-1.57 0 -1.57

Commit message: Tune sensor positions and comment the LIDAR on ergocub head

File: urdf/ergoCub/robots/ergoCubGazeboV1/model.urdf (robot description, URDF)
Before this commit: robot ergoCub, 169 links, 168 joints
Joints:
- joint r_index_dist: origin xyz=0 -0.0014998229561488108 -0.030000484918389303 rpy=3.14 0 -1.57 -> xyz=0 -0.0014998229561488108 -0.030000484918389303 rpy=0 0 0
- joint r_middle_dist: origin xyz=1.3550151000546462e-07 -0.0014995238274964628 -0.03000020325318492 rpy=3.14 0 -1.57 -> xyz=1.3550151000546462e-07 -0.0014995238274964628 -0.03000020325318492 rpy=-0.0018721728628663644 0 -2.576685250299645e-07
- joint r_thumb_dist: origin xyz=0.019999518753341633 -0.0014995177497797996 -3.909354686637556e-07 rpy=-1.57 0 -1.57 -> xyz=0.019999518753341633 -0.0014995177497797996 -3.909354686637556e-07 rpy=0 0 0
